File: lightfury_both.kicad_pcb (KiCad board)
At the start: 6 copper layers, 156.1 x 225.4 mm, 178 parts, among them U1 TLV61070ADBV, U2 SN74LV1T126DBVR

Commit message: Panelize board, generate production files. Production candidate.
Parts:
- removed the C1 at (280.4, 226.5)
- removed the C1 at (136.1, 114.5)
- removed the C2 at (275.5, 227.9)
- removed the C2 at (141.0, 113.1)
- removed the CONN1 at (269.1, 199.5)
- removed the CONN1 at (147.2, 90.6)
- removed the JST1 at (281.1, 236.5)
- removed the JST1 at (135.2, 127.6)
- removed the L1 at (278.8, 222.7)
- removed the L1 at (137.7, 118.3)
- removed the LCD1 at (269.1, 185.0)
- removed the LCD1 at (147.2, 76.1)
- removed the MCU1 at (268.6, 169.7)
- removed the MCU1 at (147.7, 60.8)
- removed the MH1 at (264.6, 46.7)
- removed the MH1 at (151.7, 155.6)
- removed the MH2 at (262.2, 128.5)
- removed the MH2 at (154.1, 237.4)
- removed the MH3 at (190.1, 148.5)
- removed the MH3 at (226.2, 39.6)
- removed the MH4 at (200.2, 39.6)
- removed the MH4 at (216.1, 148.5)
- removed the MH5 at (201.2, 138.6)
- removed the MH5 at (215.1, 247.5)
- removed the MH6 at (262.7, 258.4)
- removed the MH6 at (153.6, 149.6)
- removed the MH7 at (133.0, 133.8)
- removed the MH7 at (283.4, 242.7)
- removed the PWR1 at (132.5, 117.6)
- removed the PWR1 at (283.9, 226.5)
- removed the R1 at (141.8, 115.4)
- removed the R1 at (274.7, 225.6)
- removed the R2 at (142.5, 113.1)
- removed the R2 at (274.0, 227.9)
- removed RD1, RD10, RD11, RD12, RD13, RD14, RD2, RD3, RD4, RD5, RD6, RD7, RD8, RD9: BAV70, BAV70 SOT23
- removed the RE1 at (153.8, 111.9)
- removed the RE1 at (262.6, 220.8)
- removed RLED1: Outer Bottom, LED_WS2812B-2020_PLCC4_2.0x2.0mm
- removed RLED10, RLED11, RLED12, RLED13, RLED14, RLED16, RLED17, RLED18, RLED19, RLED2, RLED20, RLED21, RLED23, RLED25, RLED26, RLED3, RLED5, RLED6, RLED7, RLED8, RLED9: WS2812B-2020, LED_WS2812B-2020_PLCC4_2.0x2.0mm
- removed RLED15: Far Thumb, LED_WS2812B-2020_PLCC4_2.0x2.0mm
- removed RLED22: R, LED_WS2812B-2020_PLCC4_2.0x2.0mm
- removed RLED24: Inner Bottom, LED_WS2812B-2020_PLCC4_2.0x2.0mm
- removed RLED27: Inner Top, LED_WS2812B-2020_PLCC4_2.0x2.0mm
- removed RLED4: Outer Top, LED_WS2812B-2020_PLCC4_2.0x2.0mm
- removed RS1, RS10, RS11, RS12, RS13, RS14, RS15, RS16, RS17, RS18, RS19, RS2, RS20, RS21, RS22, RS23, RS24, RS25, RS26, RS27, RS3, RS4, RS5, RS6, RS7, RS8, RS9: PG1316S, PG1316S
- removed the RST1 at (160.2, 45.6)
- removed the RST1 at (256.1, 154.5)
- removed the U1 at (274.8, 222.8)
- removed the U1 at (141.7, 118.2)
- removed the U2 at (138.6, 113.9)
- removed the U2 at (277.9, 227.1)
- added C1: 10μF, Capacitor_SMD:C_0603_1608Metric, F.Cu at (153.4, 66.9)
- added C1_2: 10μF, Capacitor_SMD:C_0603_1608Metric, F.Cu at (152.6, 146.6)
- added C2: 10μF 25V, Capacitor_SMD:C_0603_1608Metric, F.Cu at (148.8, 69.2)
- added C2_2: 10μF 25V, Capacitor_SMD:C_0603_1608Metric, F.Cu at (147.5, 147.0)
- added C3: 100nF, Capacitor_SMD:C_0603_1608Metric, F.Cu at (147.3, 69.5)
- added C3_2: 100nF, Capacitor_SMD:C_0603_1608Metric, F.Cu at (146.0, 146.7)
- added C4: 10µF 25V, Capacitor_SMD:C_0603_1608Metric, F.Cu at (16.2, 31.9)
- added C4_2: 10μF 25V, Capacitor_SMD:C_0603_1608Metric, F.Cu at (115.8, 129.6)
- added C5: 10µF 25V, Capacitor_SMD:C_0603_1608Metric, F.Cu at (115.7, 79.6)
- added C5_2: 10μF 25V, Capacitor_SMD:C_0603_1608Metric, F.Cu at (17.6, 173.0)
- added CONN1: LCD HEADER, Molex_PicoBlade_53261-0871_1x08-1MP_P1.25mm_Horizontal, F.Cu at (137.2, 42.5)
- added CONN1_2: LCD HEADER, Molex_PicoBlade_53261-0871_1x08-1MP_P1.25mm_Horizontal, F.Cu at (137.2, 167.9)
- added D10_2: BAV70, BAV70 SOT23, F.Cu at (67.6, 121.9)
- added D11_2: BAV70, BAV70 SOT23, F.Cu at (86.6, 118.5)
- added D12_2: BAV70, BAV70 SOT23, F.Cu at (68.9, 115.1)
- added D13_2: BAV70, BAV70 SOT23, F.Cu at (91.2, 126.5)
- added D14_2: BAV70, BAV70 SOT23, F.Cu at (92.5, 119.6)
- added D1_2: BAV70, BAV70 SOT23, F.Cu at (73.5, 123.1)
- added D2_2: BAV70, BAV70 SOT23, F.Cu at (55.8, 119.7)
- added D3_2: BAV70, BAV70 SOT23, F.Cu at (74.8, 116.2)
- added D4_2: BAV70, BAV70 SOT23, F.Cu at (57.1, 112.8)
- added D5_2: BAV70, BAV70 SOT23, F.Cu at (79.4, 124.2)
- added D6_2: BAV70, BAV70 SOT23, F.Cu at (61.7, 120.8)
- added D7_2: BAV70, BAV70 SOT23, F.Cu at (80.7, 117.3)
- added D8_2: BAV70, BAV70 SOT23, F.Cu at (63.0, 113.9)
- added D9_2: BAV70, BAV70 SOT23, F.Cu at (85.3, 125.4)
- added JST1: Battery Connector, ceoloide:battery_connector_jst_ph_2, B.Cu at (155.9, 76.5)
- added JST1_2: Battery Connector, ceoloide:battery_connector_jst_ph_2, B.Cu at (155.9, 133.9)
- added L1: 2.2μH, huntercook:L_CJIANG_FTC404030S_4.1x4.1x3.0_SMD, F.Cu at (151.1, 63.5)
- added L1_2: 2.2μH, huntercook:L_CJIANG_FTC404030S_4.1x4.1x3.0_SMD, F.Cu at (151.7, 142.5)
- added LCD1: , LCD_1.69_Waveshare, F.Cu at (134.4, 28.2)
- added LCD1_2: , LCD_1.69_Waveshare, F.Cu at (134.4, 182.2)
- added LED10_2: WS2812B-2020, LED_WS2812B-2020_PLCC4_2.0x2.0mm, F.Cu at (90.3, 162.5)
- added LED11_2: WS2812B-2020, LED_WS2812B-2020_PLCC4_2.0x2.0mm, F.Cu at (86.7, 181.1)
- added LED12_2: WS2812B-2020, LED_WS2812B-2020_PLCC4_2.0x2.0mm, F.Cu at (83.2, 199.8)
- added LED13_2: WS2812B-2020, LED_WS2812B-2020_PLCC4_2.0x2.0mm, F.Cu at (105.6, 125.7)
- added LED14_2: WS2812B-2020, LED_WS2812B-2020_PLCC4_2.0x2.0mm, F.Cu at (126.4, 126.8)
- added LED15_2: Far Thumb, LED_WS2812B-2020_PLCC4_2.0x2.0mm, F.Cu at (146.8, 122.5)
- added LED16_2: WS2812B-2020, LED_WS2812B-2020_PLCC4_2.0x2.0mm, F.Cu at (39.1, 127.8)
- added LED17_2: WS2812B-2020, LED_WS2812B-2020_PLCC4_2.0x2.0mm, F.Cu at (34.6, 146.3)
- added LED18_2: WS2812B-2020, LED_WS2812B-2020_PLCC4_2.0x2.0mm, F.Cu at (30.0, 164.7)
- added LED19_2: WS2812B-2020, LED_WS2812B-2020_PLCC4_2.0x2.0mm, F.Cu at (25.4, 183.2)
- added LED1_2: Outer Bottom, LED_WS2812B-2020_PLCC4_2.0x2.0mm, F.Cu at (21.0, 122.0)
- added LED20_2: WS2812B-2020, LED_WS2812B-2020_PLCC4_2.0x2.0mm, F.Cu at (74.7, 143.2)
- added LED21_2: WS2812B-2020, LED_WS2812B-2020_PLCC4_2.0x2.0mm, F.Cu at (71.1, 161.8)
- added LED22_2: WS2812B-2020, LED_WS2812B-2020_PLCC4_2.0x2.0mm, F.Cu at (67.5, 180.5)
- added LED23_2: WS2812B-2020, LED_WS2812B-2020_PLCC4_2.0x2.0mm, F.Cu at (63.9, 199.1)
- added LED24_2: Inner Bottom, LED_WS2812B-2020_PLCC4_2.0x2.0mm, F.Cu at (112.8, 146.4)
- added LED25_2: WS2812B-2020, LED_WS2812B-2020_PLCC4_2.0x2.0mm, F.Cu at (109.2, 165.1)
- added LED26_2: WS2812B-2020, LED_WS2812B-2020_PLCC4_2.0x2.0mm, F.Cu at (105.6, 183.7)
- added LED27_2: Inner Top, LED_WS2812B-2020_PLCC4_2.0x2.0mm, F.Cu at (102.0, 202.4)
- added LED2_2: WS2812B-2020, LED_WS2812B-2020_PLCC4_2.0x2.0mm, F.Cu at (16.1, 140.3)
- added LED3_2: WS2812B-2020, LED_WS2812B-2020_PLCC4_2.0x2.0mm, F.Cu at (11.2, 158.7)
- added LED4_2: Outer Top, LED_WS2812B-2020_PLCC4_2.0x2.0mm, F.Cu at (6.32, 177.1)
- added LED5_2: WS2812B-2020, LED_WS2812B-2020_PLCC4_2.0x2.0mm, F.Cu at (56.7, 136.3)
- added LED6_2: WS2812B-2020, LED_WS2812B-2020_PLCC4_2.0x2.0mm, F.Cu at (52.8, 154.9)
- added LED7_2: WS2812B-2020, LED_WS2812B-2020_PLCC4_2.0x2.0mm, F.Cu at (48.9, 173.5)
- added LED8_2: WS2812B-2020, LED_WS2812B-2020_PLCC4_2.0x2.0mm, F.Cu at (44.9, 192.1)
- added LED9_2: WS2812B-2020, LED_WS2812B-2020_PLCC4_2.0x2.0mm, F.Cu at (93.9, 143.8)
- added MCU1: nice_nano, ceoloide:mcu_nice_nano, F.Cu at (131.0, 13.3)
- added MCU1_2: nice_nano, ceoloide:mcu_nice_nano, F.Cu at (131.0, 197.1)
- added MH1: , ceoloide:mounting_hole_npth, F.Cu at (13.5, 21.6)
- added MH1_2: , ceoloide:mounting_hole_npth, F.Cu at (13.5, 188.8)
- added MH2: , ceoloide:mounting_hole_npth, F.Cu at (31.4, 101.5)
- added MH2_2: , ceoloide:mounting_hole_npth, F.Cu at (31.4, 108.9)
- added MH3: , ceoloide:mounting_hole_npth, F.Cu at (49.9, 7.33)
- added MH3_2: , ceoloide:mounting_hole_npth, F.Cu at (49.9, 203.1)
- added MH4: , ceoloide:mounting_hole_npth, F.Cu at (75.5, 2.41)
- added MH4_2: , ceoloide:mounting_hole_npth, F.Cu at (75.5, 208.0)
- added MH5: , ceoloide:mounting_hole_npth, F.Cu at (93.2, 99.8)
- added MH5_2: , ceoloide:mounting_hole_npth, F.Cu at (93.2, 110.6)
- added MH6: , ceoloide:mounting_hole_npth, F.Cu at (142.0, 101.6)
- added MH6_2: , ceoloide:mounting_hole_npth, F.Cu at (142.0, 108.8)
- added MH7: , ceoloide:mounting_hole_npth, F.Cu at (159.3, 82.2)
- added MH7_2: , ceoloide:mounting_hole_npth, F.Cu at (159.3, 128.2)
- added PWR1: Power SW, ceoloide:power_switch_smd_side, F.Cu at (156.7, 66.2)
- added PWR1_2: Power SW, ceoloide:power_switch_smd_side, F.Cu at (156.7, 144.2)
- added R1: 470kΩ, Resistor_SMD:R_0603_1608Metric, F.Cu at (147.6, 67.1)
- added R1_2: 470kΩ, Resistor_SMD:R_0603_1608Metric, F.Cu at (147.2, 144.6)
- added R2: 51kΩ, Resistor_SMD:R_0603_1608Metric, F.Cu at (145.5, 68.3)
- added R2_2: 51kΩ, Resistor_SMD:R_0603_1608Metric, F.Cu at (144.5, 146.4)
- added RE1: CKW12, CKW12, F.Cu at (134.8, 64.6)
- added RE1_2: CKW12, CKW12, F.Cu at (134.8, 145.8)
- added RST1: Reset SW, ceoloide:reset_switch_smd_side, F.Cu at (115.9, 0.74)
- added RST1_2: Reset SW, ceoloide:reset_switch_smd_side, F.Cu at (115.9, 209.7)
- added S10_2: PG1316S, PG1316S, F.Cu at (53.3, 152.5)
- added S11_2: PG1316S, PG1316S, F.Cu at (49.4, 171.1)
- added S12_2: PG1316S, PG1316S, F.Cu at (45.5, 189.6)
- added S13_2: PG1316S, PG1316S, F.Cu at (75.2, 140.7)
- added S14_2: PG1316S, PG1316S, F.Cu at (71.6, 159.4)
- added S15_2: PG1316S, PG1316S, F.Cu at (68.0, 178.0)
- added S16_2: PG1316S, PG1316S, F.Cu at (64.4, 196.7)
- added S17_2: PG1316S, PG1316S, F.Cu at (94.4, 141.4)
- added S18_2: PG1316S, PG1316S, F.Cu at (90.8, 160.0)
- added S19_2: PG1316S, PG1316S, F.Cu at (87.2, 178.7)
- added S1_2: PG1316S, PG1316S, F.Cu at (21.6, 119.6)
- added S20_2: PG1316S, PG1316S, F.Cu at (83.6, 197.3)
- added S21_2: PG1316S, PG1316S, F.Cu at (113.2, 144.0)
- added S22_2: PG1316S, PG1316S, F.Cu at (109.7, 162.6)
- added S23_2: PG1316S, PG1316S, F.Cu at (106.1, 181.3)
- added S24_2: PG1316S, PG1316S, F.Cu at (102.5, 200.0)
- added S25_2: PG1316S, PG1316S, F.Cu at (106.0, 123.2)
- added S26_2: PG1316S, PG1316S, F.Cu at (126.2, 124.3)
- added S27_2: PG1316S, PG1316S, F.Cu at (146.0, 120.2)
- added S2_2: PG1316S, PG1316S, F.Cu at (16.7, 137.9)
- added S3_2: PG1316S, PG1316S, F.Cu at (11.8, 156.3)
- added S4_2: PG1316S, PG1316S, F.Cu at (6.96, 174.7)
- added S5_2: PG1316S, PG1316S, F.Cu at (39.7, 125.4)
- added S6_2: PG1316S, PG1316S, F.Cu at (35.2, 143.9)
- added S7_2: PG1316S, PG1316S, F.Cu at (30.6, 162.3)
- added S8_2: PG1316S, PG1316S, F.Cu at (26.0, 180.8)
- added S9_2: PG1316S, PG1316S, F.Cu at (57.2, 133.9)
- added U1: TLV61070ADBV, Package_TO_SOT_SMD:SOT-23-6, F.Cu at (147.1, 64.3)
- added U1_2: TLV61070ADBV, Package_TO_SOT_SMD:SOT-23-6, F.Cu at (147.8, 141.9)
- added U2: SN74LV1T126DBVR, Package_TO_SOT_SMD:SOT-23-5, F.Cu at (151.0, 67.9)
- added U2_2: SN74LV1T126DBVR, Package_TO_SOT_SMD:SOT-23-5, F.Cu at (150.1, 146.7)
- moved LED24 205.3 mm to (102.0, 7.99), turned to 10.9 degrees
- moved S24 205.0 mm to (102.5, 10.4), turned to 10.9 degrees
- moved LED23 203.1 mm to (105.6, 26.7), turned to 10.9 degrees
- moved S23 202.8 mm to (106.1, 29.1), turned to 10.9 degrees
- moved LED12 202.5 mm to (83.2, 10.6), turned to -169.1 degrees
- moved S20 202.3 mm to (83.6, 13.1), turned to 10.9 degrees
- moved LED22 201.0 mm to (109.2, 45.3), turned to 10.9 degrees
- moved S22 200.7 mm to (109.7, 47.8), turned to 10.9 degrees
- moved LED27 200.4 mm to (146.8, 87.9), turned to -19.1 degrees
- moved LED11 200.3 mm to (86.7, 29.3), turned to -169.1 degrees
- moved S19 200.1 mm to (87.2, 31.7), turned to 10.9 degrees
- moved LED20 200.1 mm to (63.9, 11.3), turned to 10.9 degrees
- moved S27 199.9 mm to (146.0, 90.2), turned to -19.1 degrees
- moved S16 199.8 mm to (64.4, 13.7), turned to 10.9 degrees
- moved LED21 198.9 mm to (112.8, 64.0), turned to 10.9 degrees
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Connections:
- net /LED_1 renamed L_/LED_1
- net /LED_10 renamed L_/LED_10
- net /LED_11 renamed L_/LED_11
- net /LED_12 renamed L_/LED_12
- net /LED_13 renamed L_/LED_13
- net /LED_14 renamed L_/LED_14
- net /LED_15 renamed L_/LED_15
- net /LED_16 renamed L_/LED_16
- net /LED_17 renamed L_/LED_17
- net /LED_18 renamed L_/LED_18
- net /LED_19 renamed L_/LED_19
- net /LED_2 renamed L_/LED_2
- net /LED_20 renamed L_/LED_20
- net /LED_21 renamed L_/LED_21
- net /LED_22 renamed L_/LED_22
- net /LED_23 renamed L_/LED_23
- net /LED_24 renamed L_/LED_24
- net /LED_25 renamed L_/LED_25
- net /LED_26 renamed L_/LED_26
- net /LED_3 renamed L_/LED_3
- net /LED_4 renamed L_/LED_4
- net /LED_5 renamed L_/LED_5
- net /LED_6 renamed L_/LED_6
- net /LED_7 renamed L_/LED_7
- net /LED_8 renamed L_/LED_8
- net /LED_9 renamed L_/LED_9
- net /far_fan renamed L_/far_fan
- net /index_bottom renamed L_/index_bottom
- net /index_home renamed L_/index_home
- net /index_num renamed L_/index_num
- net /index_top renamed L_/index_top
- net /inner_bottom renamed L_/inner_bottom
- net /inner_home renamed L_/inner_home
- net /inner_num renamed L_/inner_num
- net /inner_top renamed L_/inner_top
- net /mid_fan renamed L_/mid_fan
- net /middle_bottom renamed L_/middle_bottom
- net /middle_home renamed L_/middle_home
- net /middle_num renamed L_/middle_num
- net /middle_top renamed L_/middle_top
- net /near_fan renamed L_/near_fan
- net /outer_bottom renamed L_/outer_bottom
- net /outer_home renamed L_/outer_home
- net /outer_num renamed L_/outer_num
- net /outer_top renamed L_/outer_top
- net /pinky_bottom renamed L_/pinky_bottom
- net /pinky_home renamed L_/pinky_home
- net /pinky_num renamed L_/pinky_num
- net /pinky_top renamed L_/pinky_top
- net /ring_bottom renamed L_/ring_bottom
- net /ring_home renamed L_/ring_home
- net /ring_num renamed L_/ring_num
- net /ring_top renamed L_/ring_top
- net 5V renamed L_5V
- net C0 renamed L_C0
- net C1 renamed L_C1
- net C2 renamed L_C2
- net C3 renamed L_C3
- net C4 renamed L_C4
- net C5 renamed L_C5
- net GND renamed L_GND
- net R0 renamed L_R0
- net R1 renamed L_R1
- net R2 renamed L_R2
- net R3 renamed L_R3
- net R4 renamed L_R4
- D14 pad 2: /roller -> L_/roller
- LED1 pad 1: /LED_27 -> L_/LED_27
- LED27 pad 3: /LED_D5V -> L_/LED_D5V
Routing:
- net RAW: track 370.2 -> 0.00 mm, vias 16 -> 0
- net L_/inner_num: track 488.2 -> 245.9 mm, vias 2 -> 1
- net R_/inner_num: track 0.00 -> 242.3 mm, vias 0 -> 1
- net R_/inner_top: track 0.00 -> 240.9 mm, vias 0 -> 1
- net L_/inner_top: track 490.2 -> 249.3 mm, vias 2 -> 1
- net R_/index_num: track 0.00 -> 224.0 mm, vias 0 -> 1
- net L_/index_num: track 449.3 -> 225.3 mm, vias 2 -> 1
- net R_/index_top: track 0.00 -> 222.6 mm, vias 0 -> 1
- net L_/index_top: track 451.3 -> 228.7 mm, vias 2 -> 1
- net R_RAW: track 0.00 -> 204.5 mm, vias 0 -> 8
- net L_C2: track 394.5 -> 197.9 mm
- net R_C2: track 0.00 -> 196.6 mm
- net R_/inner_home: track 0.00 -> 193.5 mm, vias 0 -> 1
- net L_/inner_home: track 397.8 -> 204.3 mm, vias 2 -> 1
- net R_C0: track 0.00 -> 187.1 mm
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- added copper zone on In2.Cu, net R_5V
- added copper zone on In3.Cu, net R_5V
- added copper zone on B.Cu, net R_GND
- added copper zone on F.Cu, net R_GND
- added copper zone on In1.Cu, net R_GND
- added copper zone on In4.Cu, net R_GND
Other:
- board size 156.1 x 225.4 mm -> 168.2 x 217.8 mm
- rule pad_to_mask_clearance: 0.05 -> 0
